File: hardware/pcb/mini-one-pcb.kicad_pcb (KiCad board)
At the start: 4 copper layers, 50 x 70 mm, 120 parts, among them J1 ~{RUN}, J10 PYRO3, J11 MSD-1-A, J12 SMA_Edge, J13 SMA_Edge, J2 ~{SS}, J3 XT30-V-M, J4 USB1030, J5 PYRO1, J6 SERVO1, J7 SERVO2, J8 PYRO2, J9 PYRO ARM, Q1 AO3400A, Q2 AO3400A, Q3 AO3400A, U1 RP2354B, U2 AMS1117-3.3, U3 BMP585, U4 W25Q128JVSIQ, U5 LSM6DSV320XTR, U6 MAX-M10S, U7 RAK3172-8-SM-NI, Y1 ABM8-272-T3

Commit message: Revision 1 on layout editor and adding reference images
Routing:
- net GND: vias 296 -> 295
Changed lines of the file:
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@@
-	)
-	(via
-		(at 135.2 68.6)
-		(size 0.45)
-		(drill 0.2)
-		(layers "F.Cu" "B.Cu")
-		(free yes)
-		(net "GND")
 	)
 	(via
