File: hardware/pcb/mini-one-pcb.kicad_pcb (KiCad board)
At the start: 4 copper layers, 50 x 70 mm, 120 parts, among them J1 ~{RUN}, J10 PYRO3, J11 MSD-1-A, J12 SMA_Edge, J13 SMA_Edge, J2 ~{SS}, J3 XT30-V-M, J4 USB1030, J5 PYRO1, J6 SERVO1, J7 SERVO2, J8 PYRO2, J9 PYRO ARM, Q1 AO3400A, Q2 AO3400A, Q3 AO3400A, U1 RP2354B, U2 AMS1117-3.3, U3 BMP585, U4 W25Q128JVSIQ, U5 LSM6DSV320XTR, U6 MAX-M10S, U7 RAK3172-8-SM-NI, Y1 ABM8-272-T3

Commit message: PCB Rev 2
Parts:
- removed TP1: +1.1V, TestPoint:TestPoint_Pad_D2.5mm
- removed TP2: VBUS, TestPoint:TestPoint_Pad_D2.5mm
- removed TP3: +3.3V, TestPoint:TestPoint_Pad_D2.5mm
- removed TP4: GND, TestPoint:TestPoint_Pad_D2.5mm
- added C32: 470u, Capacitor_THT:CP_Radial_D8.0mm_P3.50mm, F.Cu at (125.8, 103.0)
- added G***: QR_Kestrel_Repo_14mm, mini-one-footprint-lib:QR_Kestrel_Repo_14mm, B.Cu at (120.0, 88.0)
- added G***: Warning_Knockout_3mm, mini-one-footprint-lib:Warning_Knockout_3mm, B.Cu at (134.0, 53.0)
- added G***: Warning_Knockout_3mm, mini-one-footprint-lib:Warning_Knockout_3mm, B.Cu at (109.7, 116.5)
- added G***: Warning_Knockout_3mm, mini-one-footprint-lib:Warning_Knockout_3mm, B.Cu at (106.0, 60.1)
- added G***: Kestrel_FC_Logo_P3, mini-one-footprint-lib:Kestrel_FC_Logo_P3, B.Cu at (120.0, 75.0)
- U5: value LSM6DSV320XTR -> LSM6DSV32X
- moved R2 8.96 mm to (110.4, 66.4)
- moved J2 8.96 mm to (111.0, 68.4), turned to 180 degrees
- moved C20 1.61 mm to (123.6, 67.4)
- moved C21 1.61 mm to (124.8, 67.4)
- renumbered C32 to C33, C33 to C34, C34 to C35, C35 to C36, C36 to C37, C37 to C38, C40 to C39, C38 to C40, C39 to C42, C42 to C43, C43 to C44, C44 to C45, C45 to C46, C46 to C47, R29 to R26, R30 to R27, R26 to R28, R27 to R29, R28 to R30
Routing:
- net +1.1V: track 30.5 -> 8.30 mm, vias 1 -> 0
- net VBUS: track 12.9 -> 0.00 mm, vias 0 -> 9
- net Net-(J2-Pin_1): track 5.31 -> 14.2 mm
- net GND: track 14.8 -> 12.2 mm, vias 295 -> 254
- net USB_D+: track 23.6 -> 20.9 mm, vias 1 -> 0
- net +3.3V: track 32.6 -> 30.0 mm, vias 44 -> 39
- net Net-(J1-Pin_2): track 9.91 -> 10.9 mm
- net SPI0_MISO: track 12.8 -> 13.7 mm
- net USB_D-: track 20.5 -> 20.9 mm, vias 1 -> 0
- net +BATT: vias 12 -> 8
- added copper zone on B.Cu, net VBUS
- added copper zone on In2.Cu, net VBUS
Other:
- board text added: "2S LiPo/LiFe"
- board text added: "DO NOT CONNECT USB WHILE BATT CONNECTED"
- board text added: "LoRa: ATTACH ANT BEFORE POWER-ON"
- board text added: "STATUS A"
- board text added: "STATUS B"
- board text added: "STATUS C"
- board text removed: "2S LiFe IN"
- board text removed: "5V0"
- board text removed: "A"
- board text removed: "B"
- board text removed: "C"
- board text removed: "Edward S. 2026"
- board text removed: "GND"
- board text removed: "TEST POINTS"
- board text removed: "WARNING Do not power the board without any antennas connected!"
