File: hardware/pcb/RF.kicad_sch (KiCad schematic)
At the start: 13 parts, among them J12 SMA_Edge, J13 SMA_Edge, U6 MAX-M10S, U7 RAK3172-8-SM-NI

Commit message: PCB Rev 2
Parts:
- removed TP3: +3.3V, TestPoint:TestPoint_Pad_D2.5mm, symbol PCM_4ms_Connector:TestPoint
- renumbered C42 to C43, C43 to C44, C44 to C45, C45 to C46, C46 to C47
Changed lines of the file:
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@@
-	(wire
-		(pts
-			(xy 161.29 182.88) (xy 162.56 182.88)
-		)
-		(stroke
-			(width 0)
-			(type default)
-		)
-	)
 	(wire
 		(pts
@@
 		(in_pos_files yes)
 		(dnp no)
-		(property "Reference" "C43"
+		(property "Reference" "C44"
 			(at 140.208 118.364 0)
 			(show_name no)
@@
 			(project "mini-one-pcb"
 				(path "/ceb43049-5cbf-4c56-aa0a-c2184d7e2ca1/755120ff-6313-4b41-b2ec-5703ee420036"
-					(reference "C43")
+					(reference "C44")
 					(unit 1)
 				)
@@
 		(in_pos_files yes)
 		(dnp no)
-		(property "Reference" "C46"
+		(property "Reference" "C47"
 			(at 151.13 36.83 0)
 			(show_name no)
@@
 			(project "mini-one-pcb"
 				(path "/ceb43049-5cbf-4c56-aa0a-c2184d7e2ca1/755120ff-6313-4b41-b2ec-5703ee420036"
-					(reference "C46")
+					(reference "C47")
 					(unit 1)
 				)
@@
 		(in_pos_files yes)
 		(dnp no)
-		(property "Reference" "#PWR075"
+		(property "Reference" "#PWR076"
 			(at 102.87 127 0)
 			(hide yes)
@@
 			(project "mini-one-pcb"
 				(path "/ceb43049-5cbf-4c56-aa0a-c2184d7e2ca1/755120ff-6313-4b41-b2ec-5703ee420036"
-					(reference "#PWR075")
+					(reference "#PWR076")
 					(unit 1)
 				)
@@
 		(dnp no)
 		(fields_autoplaced yes)
-		(property "Reference" "#PWR084"
+		(property "Reference" "#PWR085"
 			(at 154.94 143.51 0)
 			(hide yes)
@@
 			(project "mini-one-pcb"
 				(path "/ceb43049-5cbf-4c56-aa0a-c2184d7e2ca1/755120ff-6313-4b41-b2ec-5703ee420036"
-					(reference "#PWR084")
+					(reference "#PWR085")
 					(unit 1)
 				)
@@
 		(in_pos_files yes)
 		(dnp no)
-		(property "Reference" "#PWR080"
+		(property "Reference" "#PWR081"
 			(at 146.05 118.11 0)
 			(hide yes)
@@
 			(project "mini-one-pcb"
 				(path "/ceb43049-5cbf-4c56-aa0a-c2184d7e2ca1/755120ff-6313-4b41-b2ec-5703ee420036"
-					(reference "#PWR080")
+					(reference "#PWR081")
 					(unit 1)
 				)
@@
 		(in_pos_files yes)
 		(dnp no)
-		(property "Reference" "C42"
+		(property "Reference" "C43"
 			(at 130.81 36.83 0)
 			(show_name no)
@@
 			(project "mini-one-pcb"
 				(path "/ceb43049-5cbf-4c56-aa0a-c2184d7e2ca1/755120ff-6313-4b41-b2ec-5703ee420036"
-					(reference "C42")
+					(reference "C43")
 					(unit 1)
 				)
@@
 		(dnp no)
 		(fields_autoplaced yes)
-		(property "Reference" "#PWR079"
+		(property "Reference" "#PWR080"
 			(at 144.78 73.66 0)
 			(hide yes)
@@
 			(project "mini-one-pcb"
 				(path "/ceb43049-5cbf-4c56-aa0a-c2184d7e2ca1/755120ff-6313-4b41-b2ec-5703ee420036"
-					(reference "#PWR079")
+					(reference "#PWR080")
 					(unit 1)
 				)
@@
 		(dnp no)
 		(fields_autoplaced yes)
-		(property "Reference" "#PWR076"
+		(property "Reference" "#PWR077"
 			(at 102.87 152.4 0)
 			(hide yes)
@@
 			(project "mini-one-pcb"
 				(path "/ceb43049-5cbf-4c56-aa0a-c2184d7e2ca1/755120ff-6313-4b41-b2ec-5703ee420036"
-					(reference "#PWR076")
+					(reference "#PWR077")
 					(unit 1)
 				)
@@
 		(in_pos_files yes)
 		(dnp no)
-		(property "Reference" "C45"
+		(property "Reference" "C46"
 			(at 150.368 118.364 0)
 			(show_name no)
@@
 			(project "mini-one-pcb"
 				(path "/ceb43049-5cbf-4c56-aa0a-c2184d7e2ca1/755120ff-6313-4b41-b2ec-5703ee420036"
-					(reference "C45")
+					(reference "C46")
 					(unit 1)
 				)
@@
 		(dnp no)
 		(fields_autoplaced yes)
-		(property "Reference" "#PWR081"
+		(property "Reference" "#PWR082"
 			(at 146.05 130.81 0)
 			(hide yes)
@@
 			(project "mini-one-pcb"
 				(path "/ceb43049-5cbf-4c56-aa0a-c2184d7e2ca1/755120ff-6313-4b41-b2ec-5703ee420036"
-					(reference "#PWR081")
+					(reference "#PWR082")
 					(unit 1)
 				)
@@
 		(dnp no)
 		(fields_autoplaced yes)
-		(property "Reference" "#PWR083"
+		(property "Reference" "#PWR084"
 			(at 148.59 49.53 0)
 			(hide yes)
@@
 			(project "mini-one-pcb"
 				(path "/ceb43049-5cbf-4c56-aa0a-c2184d7e2ca1/755120ff-6313-4b41-b2ec-5703ee420036"
-					(reference "#PWR083")
+					(reference "#PWR084")
 					(unit 1)
 				)
@@
 		(in_pos_files yes)
 		(dnp no)
-		(property "Reference" "#PWR082"
+		(property "Reference" "#PWR083"
 			(at 148.59 36.83 0)
 			(hide yes)
@@
 			(project "mini-one-pcb"
 				(path "/ceb43049-5cbf-4c56-aa0a-c2184d7e2ca1/755120ff-6313-4b41-b2ec-5703ee420036"
-					(reference "#PWR082")
+					(reference "#PWR083")
 					(unit 1)
 				)
@@
 		(dnp no)
 		(fields_autoplaced yes)
-		(property "Reference" "#PWR077"
+		(property "Reference" "#PWR078"
 			(at 128.27 88.9 0)
 			(hide yes)
@@
 			(project "mini-one-pcb"
 				(path "/ceb43049-5cbf-4c56-aa0a-c2184d7e2ca1/755120ff-6313-4b41-b2ec-5703ee420036"
-					(reference "#PWR077")
+					(reference "#PWR078")
 					(unit 1)
 				)
@@
 		(dnp no)
 		(fields_autoplaced yes)
-		(property "Reference" "#PWR078"
+		(property "Reference" "#PWR079"
 			(at 132.08 191.77 0)
 			(hide yes)
@@
 			(project "mini-one-pcb"
 				(path "/ceb43049-5cbf-4c56-aa0a-c2184d7e2ca1/755120ff-6313-4b41-b2ec-5703ee420036"
-					(reference "#PWR078")
+					(reference "#PWR079")
 					(unit 1)
 				)
@@
 		(in_pos_files yes)
 		(dnp no)
-		(property "Reference" "#PWR074"
+		(property "Reference" "#PWR075"
 			(at 95.25 67.31 0)
 			(hide yes)
@@
 			(project "mini-one-pcb"
 				(path "/ceb43049-5cbf-4c56-aa0a-c2184d7e2ca1/755120ff-6313-4b41-b2ec-5703ee420036"
-					(reference "#PWR074")
+					(reference "#PWR075")
 					(unit 1)
 				)
@@
 		(in_pos_files yes)
 		(dnp no)
-		(property "Reference" "C44"
+		(property "Reference" "C45"
 			(at 140.97 36.83 0)
 			(show_name no)
@@
 			(project "mini-one-pcb"
 				(path "/ceb43049-5cbf-4c56-aa0a-c2184d7e2ca1/755120ff-6313-4b41-b2ec-5703ee420036"
-					(reference "C44")
+					(reference "C45")
 					(unit 1)
 				)
-			)
-		)
-	)
-	(symbol
-		(lib_id "power:+3.3V")
-		(at 161.29 182.88 90)
-		(unit 1)
-		(body_style 1)
-		(exclude_from_sim no)
-		(in_bom yes)
-		(on_board yes)
-		(in_pos_files yes)
-		(dnp no)
-		(property "Reference" "#PWR085"
-			(at 165.1 182.88 0)
-			(hide yes)
-			(show_name no)
-			(do_not_autoplace no)
-			(effects
-				(font
-					(size 1.27 1.27)
-				)
-			)
-		)
-		(property "Value" "+3.3V"
-			(at 155.702 182.88 90)
-			(show_name no)
-			(do_not_autoplace no)
-			(effects
-				(font
-					(size 1.27 1.27)
-				)
-			)
-		)
-		(property "Footprint" ""
-			(at 161.29 182.88 0)
-			(hide yes)
-			(show_name no)
-			(do_not_autoplace no)
-			(effects
-				(font
-					(size 1.27 1.27)
-				)
-			)
-		)
-		(property "Datasheet" ""
-			(at 161.29 182.88 0)
-			(hide yes)
-			(show_name no)
-			(do_not_autoplace no)
-			(effects
-				(font
-					(size 1.27 1.27)
-				)
-			)
-		)
-		(property "Description" "Power symbol creates a global label with name \"+3.3V\""
-			(at 161.29 182.88 0)
-			(hide yes)
-			(show_name no)
-			(do_not_autoplace no)
-			(effects
-				(font
-					(size 1.27 1.27)
-				)
-			)
-		)
-		(pin "1"
-		)
-		(instances
-			(project "mini-one-pcb"
-				(path "/ceb43049-5cbf-4c56-aa0a-c2184d7e2ca1/755120ff-6313-4b41-b2ec-5703ee420036"
-					(reference "#PWR085")
-					(unit 1)
-				)
-			)
-		)
-	)
-	(symbol
-		(lib_id "PCM_4ms_Connector:TestPoint")
-		(at 162.56 182.88 270)
-		(unit 1)
-		(body_style 1)
-		(exclude_from_sim no)
-		(in_bom yes)
-		(on_board yes)
-		(in_pos_files yes)
-		(dnp yes)
-		(property "Reference" "TP3"
-			(at 171.323 184.277 90)
-			(show_name no)
-			(do_not_autoplace no)
-			(effects
-				(font
-					(size 1.27 1.27)
-				)
-				(justify right)
-			)
-		)
-		(property "Value" "+3.3V"
-			(at 172.593 181.737 90)
-			(show_name no)
-			(do_not_autoplace no)
-			(effects
-				(font
-					(size 1.27 1.27)
-				)
-				(justify right)
-			)
-		)
-		(property "Footprint" "TestPoint:TestPoint_Pad_D2.5mm"
-			(at 162.56 187.96 0)
-			(hide yes)
-			(show_name no)
-			(do_not_autoplace no)
-			(effects
-				(font
-					(size 1.27 1.27)
-				)
-			)
-		)
-		(property "Datasheet" ""
-			(at 162.56 187.96 0)
-			(hide yes)
-			(show_name no)
-			(do_not_autoplace no)
-			(effects
-				(font
-					(size 1.27 1.27)
-				)
-			)
-		)
-		(property "Description" "test point"
-			(at 162.56 182.88 0)
-			(hide yes)
-			(show_name no)
-			(do_not_autoplace no)
-			(effects
-				(font
-					(size 1.27 1.27)
-				)
-			)
-		)
-		(pin "1"
-		)
-		(instances
-			(project "mini-one-pcb"
-				(path "/ceb43049-5cbf-4c56-aa0a-c2184d7e2ca1/755120ff-6313-4b41-b2ec-5703ee420036"
-					(reference "TP3")
-					(unit 1)
-				)
