File: hardware/pcb/outputs.kicad_sch (KiCad schematic)
At the start: 33 parts, among them J10 PYRO3, J5 PYRO1, J6 SERVO1, J7 SERVO2, J8 PYRO2, J9 PYRO ARM, Q1 AO3400A, Q2 AO3400A, Q3 AO3400A

Commit message: PCB Rev 2
Parts:
- added C32: 470u, Capacitor_THT:CP_Radial_D8.0mm_P3.50mm, symbol Device:C_Polarized
- renumbered C32 to C33, C33 to C34
Connections:
- net +BATT: now also C32.1
- net GND: now also C32.2
