File: hardware/pcb/sensors-and-memory.kicad_sch (KiCad schematic)
At the start: 22 parts, among them J11 MSD-1-A, U3 BMP585, U4 W25Q128JVSIQ, U5 LSM6DSV32X

Commit message: PCB Rev 2
Parts:
- renumbered C34 to C35, C35 to C36, C36 to C37, C37 to C38, C40 to C39, C38 to C40, C39 to C42, R29 to R26, R30 to R27, R26 to R28, R27 to R29, R28 to R30
